Commit message: finalizando xacro

File: urdf/softsnake.xacro (robot description, xacro)
@@ -83,3 +83,39 @@
         <origin rpy="0 0 0" xyz="0 0 0.0125"/>
     </joint>
+     <link name="joint2_link">
+        <visual>
+            <geometry>
+                <box size = "0.07 0.015 0.18"/>
+            </geometry>
+        <material name="silver">
+            <color rgba="0.75 0.75 0.75 1"/>
+        </material>
+        <origin rpy="0 0 0" xyz="0 0 0.08"/>
+        </visual>
+    </link>
+    <joint name="joint2_link" type="revolute">
+        <axis xyz="1 0 0"/>
+        <parent link="joint1_link"/>
+        <child link="joint2_link"/>
+        <limit effort="30" velocity="1.0" lower="-1.5" upper="1.5" />
+        <origin rpy="0 0 0" xyz="0 0 0.14"/>
+    </joint>
+    <link name="joint3_link">
+        <visual>
+            <geometry>
+                <box size = "0.07 0.015 0.065"/>
+            </geometry>
+        <material name="silver">
+            <color rgba="0.75 0.75 0.75 1"/>
+        </material>
+        <origin rpy="0 0 0" xyz="0 0 0.025"/>
+        </visual>
+    </link>
+    <joint name="joint3_link" type="revolute">
+        <axis xyz="1 0 0"/>
+        <parent link="joint2_link"/>
+        <child link="joint3_link"/>
+        <limit effort="30" velocity="1.0" lower="-1.5" upper="1.5" />
+        <origin rpy="0 0 0" xyz="0 0 0.15"/>
+    </joint>
 </robot>
